File: PCB/TImeDelaySafe/TImeDelaySafe.sch (KiCad schematic (older format))
At the start: 13 parts, among them M1 UnlockMotor, Q1 K\\N2222A, SW1 HomeSensor, SW2 LockButton, SW3 OpenButton, U1 PICAXEM2

Commit message: ready to test
Parts:
- Q1: value K\\N2222A -> KN2222A
- R1: value 4k7 -> 390
Changed lines of the file:
@@
 P 6800 3200
 F 0 "Q1" H 6991 3246 50  0000 L CNN
-F 1 "K\\N2222A" H 6991 3155 50  0000 L CNN
+F 1 "KN2222A" H 6991 3155 50  0000 L CNN
 F 2 "Package_TO_SOT_THT:TO-92_Inline" H 7000 3125 50  0001 L CIN
 F 3 "http://www.fairchildsemi.com/ds/PN/PN2222A.pdf" H 6800 3200 50  0001 L CNN
@@
 P 6250 1750
 F 0 "R1" H 6182 1704 50  0000 R CNN
-F 1 "4k7" H 6182 1795 50  0000 R CNN
+F 1 "390" H 6182 1795 50  0000 R CNN
 F 2 "" V 6290 1740 50  0001 C CNN
 F 3 "~" H 6250 1750 50  0001 C CNN
